File: KiCAD/RFID.kicad_sch (KiCad schematic)
At the start: 56 parts, among them J1 JST SH Con, J3 Display Connector, J5 Battery Conenctor, SW2 RUN, SW4 A_BTN, SW5 B_BTN, U1 RP2040, Y2 12M

Commit message: Corrected wrong battery footprint orientation
Connections:
- net Battery Gauge/BAT: now also J5.3 (Pin_3); no longer J5.1 (Pin_1)
Changed lines of the file:
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@@
 	)
 	(junction
-		(at 97.79 35.56)
-		(diameter 0)
-		(color 0 0 0 0)
-	)
-	(junction
 		(at 39.37 147.32)
 		(diameter 0)
@@
 	)
 	(junction
+		(at 97.79 35.56)
+		(diameter 0)
+		(color 0 0 0 0)
+	)
+	(junction
 		(at 67.31 76.2)
 		(diameter 0)
@@
 	)
 	(no_connect
-		(at 92.71 40.64)
-	)
-	(no_connect
 		(at 102.87 137.16)
 	)
@@
 	)
 	(no_connect
+		(at 92.71 40.64)
+	)
+	(no_connect
 		(at 102.87 127)
 	)
@@
 	(wire
 		(pts
+			(xy 92.71 35.56) (xy 97.79 35.56)
+		)
+		(stroke
+			(width 0)
+			(type default)
+		)
+	)
+	(wire
+		(pts
 			(xy 50.8 157.48) (xy 52.07 157.48)
 		)
@@
 	(wire
 		(pts
-			(xy 92.71 35.56) (xy 97.79 35.56)
-		)
-		(stroke
-			(width 0)
-			(type default)
-		)
-	)
-	(wire
-		(pts
 			(xy 44.45 106.68) (xy 46.99 106.68)
 		)
@@
 		(lib_id "Connector:Conn_01x03_Pin")
 		(at 87.63 38.1 0)
+		(mirror x)
 		(unit 1)
 		(body_style 1)
@@
 		(in_pos_files yes)
 		(dnp no)
-		(fields_autoplaced yes)
 		(property "Reference" "J5"
-			(at 88.265 30.48 0)
+			(at 86.868 29.21 0)
 			(show_name no)
 			(do_not_autoplace no)
@@
 		)
 		(property "Value" "Battery Conenctor"
-			(at 88.265 33.02 0)
+			(at 86.868 31.75 0)
 			(show_name no)
 			(do_not_autoplace no)
