File: KiCAD/Power_sw.kicad_sch (KiCad schematic)
At the start: 15 parts, among them IC2 BQ24075TRGTT

Commit message: Added everything for ordering
Parts:
- R1: value 46k8 -> 46k4
Other:
- note added: "Replace and cheack R6, R5, R1 and TH1 values with the BQ24075'sdatasheet"
- note removed: "Replace and cheack R6, R5, R1 and TH1 values with the BQ24075'sdatasheet (use claude to help)"
Changed lines of the file:
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@@
 		)
 	)
-	(text "Replace and cheack R6, R5, R1 and TH1 values \nwith the BQ24075'sdatasheet (use claude to help)\n"
+	(text "Replace and cheack R6, R5, R1 and TH1 values \nwith the BQ24075'sdatasheet"
 		(exclude_from_sim no)
 		(at 140.97 45.72 0)
@@
 			)
 		)
-		(property "Value" "46k8"
+		(property "Value" "46k4"
 			(at 154.94 54.6099 0)
 			(show_name no)
